Commit message: color & skid steering

File: udacity_bot/urdf/udacity_bot.xacro (robot description, xacro)
@@ -1,4 +1,20 @@
 <?xml version='1.0'?>
 <robot name="udacity_bot" xmlns:xacro="http://www.ros.org/wiki/xacro">
+  <!-- Color descriptions -->
+  <material name="orange">
+    <color rgba="1 0.5 0.32 1"/>
+  </material>
+  <material name="black">
+    <color rgba="0 0 0 1"/>
+  </material>
+  <material name="white">
+    <color rgba="1 1 1 1"/>
+  </material>
+  <material name="gray">
+    <color rgba="0.8 0.8 0.8 1"/>
+  </material>
+  <material name="blue">
+    <color rgba="0 0 1 1"/>
+  </material>
   <xacro:include filename="$(find udacity_bot)/urdf/udacity_bot.gazebo" />
   <link name="robot_footprint"></link>
@@ -30,31 +46,8 @@
         <box size=".4 .2 .1"/>
       </geometry>
-    </visual>
-    <collision name='back_caster_collision'>
-      <origin xyz="-0.15 0 -0.05" rpy=" 0 0 0"/>
-      <geometry>
-        <sphere radius="0.0499"/>
-      </geometry>
-    </collision>
-    <visual name='back_caster_visual'>
-      <origin xyz="-0.15 0 -0.05" rpy=" 0 0 0"/>
-      <geometry>
-        <sphere radius="0.05"/>
-      </geometry>
-    </visual>
-    <collision name='front_caster_collision'>
-      <origin xyz="0.15 0 -0.05" rpy=" 0 0 0"/>
-      <geometry>
-        <sphere radius="0.0499"/>
-      </geometry>
-    </collision>
-    <visual name='front_caster_visual'>
-      <origin xyz="0.15 0 -0.05" rpy=" 0 0 0"/>
-      <geometry>
-        <sphere radius="0.05"/>
-      </geometry>
+      <material name="blue"/>
     </visual>
   </link>
-  <link name='left_wheel'>
+  <link name='left_front_wheel'>
     <inertial>
       <mass value="5.0"/>
@@ -77,9 +70,10 @@
         <cylinder radius="0.1" length="0.05"/>
       </geometry>
+      <material name="black"/>
     </visual>
   </link>
-  <joint type="continuous" name="left_wheel_hinge">
-      <origin xyz="0 0.15 0" rpy="0 0 0"/>
-      <child link="left_wheel"/>
+  <joint type="continuous" name="left_front_wheel_hinge">
+      <origin xyz="0.15 0.15 0" rpy="0 0 0"/>
+      <child link="left_front_wheel"/>
       <parent link="chassis"/>
       <axis xyz="0 1 0" rpy="0 0 0"/>
@@ -87,5 +81,5 @@
       <dynamics damping="1.0" friction="1.0"/>
    </joint>
-   <link name='right_wheel'>
+   <link name='right_front_wheel'>
      <inertial>
        <mass value="5.0"/>
@@ -108,9 +102,10 @@
          <cylinder radius="0.1" length="0.05"/>
        </geometry>
+       <material name="black"/>
      </visual>
    </link>
-   <joint type="continuous" name="right_wheel_hinge">
-       <origin xyz="0 -0.15 0" rpy="0 0 0"/>
-       <child link="right_wheel"/>
+   <joint type="continuous" name="right_front_wheel_hinge">
+       <origin xyz="0.15 -0.15 0" rpy="0 0 0"/>
+       <child link="right_front_wheel"/>
        <parent link="chassis"/>
        <axis xyz="0 1 0" rpy="0 0 0"/>
@@ -118,4 +113,68 @@
        <dynamics damping="1.0" friction="1.0"/>
     </joint>
+    <link name='left_back_wheel'>
+      <inertial>
+        <mass value="5.0"/>
+        <origin xyz="0.0 0 0" rpy=" 0 1.5707 1.5707"/>
+        <inertia
+            ixx="0.1" ixy="0" ixz="0"
+            iyy="0.1" iyz="0"
+            izz="0.1"
+        />
+      </inertial>
+      <collision name='collision'>
+        <origin xyz="0 0 0" rpy=" 0 1.5707 1.5707"/>
+        <geometry>
+          <cylinder radius="0.1" length="0.05"/>
+        </geometry>
+      </collision>
+      <visual name='visual'>
+        <origin xyz="0 0 0" rpy=" 0 1.5707 1.5707"/>
+        <geometry>
+          <cylinder radius="0.1" length="0.05"/>
+        </geometry>
+        <material name="black"/>
+      </visual>
+    </link>
+    <joint type="continuous" name="left_back_wheel_hinge">
+        <origin xyz="-0.15 0.15 0" rpy="0 0 0"/>
+        <child link="left_back_wheel"/>
+        <parent link="chassis"/>
+        <axis xyz="0 1 0" rpy="0 0 0"/>
+        <limit effort="10000" velocity="1000"/>
+        <dynamics damping="1.0" friction="1.0"/>
+     </joint>
+     <link name='right_back_wheel'>
+       <inertial>
+         <mass value="5.0"/>
+         <origin xyz="0.0 0 0" rpy=" 0 1.5707 1.5707"/>
+         <inertia
+             ixx="0.1" ixy="0" ixz="0"
+             iyy="0.1" iyz="0"
+             izz="0.1"
+         />
+       </inertial>
+       <collision name='collision'>
+         <origin xyz="0 0 0" rpy=" 0 1.5707 1.5707"/>
+         <geometry>
+           <cylinder radius="0.1" length="0.05"/>
+         </geometry>
+       </collision>
+       <visual name='visual'>
+         <origin xyz="0 0 0" rpy=" 0 1.5707 1.5707"/>
+         <geometry>
+           <cylinder radius="0.1" length="0.05"/>
+         </geometry>
+         <material name="black"/>
+       </visual>
+     </link>
+     <joint type="continuous" name="right_back_wheel_hinge">
+         <origin xyz="-0.15 -0.15 0" rpy="0 0 0"/>
+         <child link="right_back_wheel"/>
+         <parent link="chassis"/>
+         <axis xyz="0 1 0" rpy="0 0 0"/>
+         <limit effort="10000" velocity="1000"/>
+         <dynamics damping="1.0" friction="1.0"/>
+      </joint>
     <!-- Camera link -->
     <link name="camera">
@@ -140,4 +199,5 @@
             <box size="0.05 0.05 0.05" />
         </geometry>
+        <material name="gray"/>
      </visual>
    </link>

Commit message: add in color property

File: udacity_bot/urdf/udacity_bot.xacro (robot description, xacro)
@@ -1,11 +1,19 @@
 <?xml version='1.0'?>
 <robot name="udacity_bot" xmlns:xacro="http://www.ros.org/wiki/xacro">
+  <!-- Color descriptions -->
+  <material name="blue">
+    <color rgba="0 0 0.8 1"/>
+  </material>
+  <material name="black">
+    <color rgba="0 0 0 1"/>
+  </material>
+  <material name="white">
+    <color rgba="1 1 1 1"/>
+  </material>
+  <material name="green">
+    <color rgba="0 1 0 1"/>
+  </material>
   <xacro:include filename="$(find udacity_bot)/urdf/udacity_bot.gazebo" />
   <link name="robot_footprint"></link>
-  <joint name="robot_footprint_joint" type="fixed">
-    <origin xyz="0 0 0" rpy="0 0 0" />
-    <parent link="robot_footprint"/>
-    <child link="chassis" />
-  </joint>
   <link name='chassis'>
     <pose>0 0 0.1 0 0 0</pose>
@@ -30,4 +38,5 @@
         <box size=".4 .2 .1"/>
       </geometry>
+      <material name="blue"/>
     </visual>
     <collision name='back_caster_collision'>
@@ -56,4 +65,9 @@
     </visual>
   </link>
+  <joint name="robot_footprint_joint" type="fixed">
+    <origin xyz="0 0 0" rpy="0 0 0" />
+    <parent link="robot_footprint"/>
+    <child link="chassis" />
+  </joint>
   <link name='left_wheel'>
     <inertial>
@@ -72,9 +86,10 @@
       </geometry>
     </collision>
-    <visual name='visual'>
+    <visual>
       <origin xyz="0 0 0" rpy=" 0 1.5707 1.5707"/>
       <geometry>
         <cylinder radius="0.1" length="0.05"/>
       </geometry>
+      <material name="black"/>
     </visual>
   </link>
@@ -103,9 +118,10 @@
        </geometry>
      </collision>
-     <visual name='visual'>
+     <visual>
        <origin xyz="0 0 0" rpy=" 0 1.5707 1.5707"/>
        <geometry>
          <cylinder radius="0.1" length="0.05"/>
        </geometry>
+       <material name="black"/>
      </visual>
    </link>
@@ -135,9 +151,10 @@
         </geometry>
         </collision>
-    <visual name="visual">
+    <visual>
         <origin xyz="0 0 0" rpy="0 0 0"/>
         <geometry>
             <box size="0.05 0.05 0.05" />
         </geometry>
+        <material name="green"/>
      </visual>
    </link>
