Commit message: rename 4wd bot to rover_bot

File: rover_bot/urdf/rover_bot.xacro (robot description, xacro)
@@ -1,4 +1,4 @@
 <?xml version='1.0'?>
-<robot name="udacity_bot" xmlns:xacro="http://www.ros.org/wiki/xacro">
+<robot name="rover_bot" xmlns:xacro="http://www.ros.org/wiki/xacro">
   <!-- Color descriptions -->
   <material name="blue">
@@ -14,5 +14,5 @@
     <color rgba="0 1 0 1"/>
   </material>
-  <xacro:include filename="$(find udacity_bot)/urdf/udacity_bot.gazebo" />
+  <xacro:include filename="$(find rover_bot)/urdf/rover_bot.gazebo" />
   <link name="robot_footprint"></link>
   <link name='chassis'>
@@ -225,6 +225,6 @@
            <origin xyz="0 0 0" rpy="0 0 0"/>
            <geometry>
-               <mesh filename="package://udacity_bot/meshes/hokuyo.dae"/>
-               <!-- mesh filename="$(find udacity_bot)/meshes/hokuyo.dae"/ -->
+               <mesh filename="package://rover_bot/meshes/hokuyo.dae"/>
+               <!-- mesh filename="$(find rover_bot)/meshes/hokuyo.dae"/ -->
            </geometry>
         </visual>

Commit message: reduce wheel distance

File: rover_bot/urdf/rover_bot.xacro (robot description, xacro)
@@ -71,5 +71,5 @@
   </link>
   <joint type="continuous" name="left_front_wheel_hinge">
-      <origin xyz="0.15 0.15 0" rpy="0 0 0"/>
+      <origin xyz="0.125 0.15 0" rpy="0 0 0"/>
       <child link="left_front_wheel"/>
       <parent link="chassis"/>
@@ -103,5 +103,5 @@
    </link>
    <joint type="continuous" name="right_front_wheel_hinge">
-       <origin xyz="0.15 -0.15 0" rpy="0 0 0"/>
+       <origin xyz="0.125 -0.15 0" rpy="0 0 0"/>
        <child link="right_front_wheel"/>
        <parent link="chassis"/>
@@ -135,5 +135,5 @@
     </link>
     <joint type="continuous" name="left_back_wheel_hinge">
-        <origin xyz="-0.15 0.15 0" rpy="0 0 0"/>
+        <origin xyz="-0.125 0.15 0" rpy="0 0 0"/>
         <child link="left_back_wheel"/>
         <parent link="chassis"/>
@@ -167,5 +167,5 @@
      </link>
      <joint type="continuous" name="right_back_wheel_hinge">
-         <origin xyz="-0.15 -0.15 0" rpy="0 0 0"/>
+         <origin xyz="-0.125 -0.15 0" rpy="0 0 0"/>
          <child link="right_back_wheel"/>
          <parent link="chassis"/>
